Commit message: minimum vis

File: urdf/kettle.urdf (robot description, URDF)
Before this commit: robot kettle, 4 links, 3 joints
Links:
- link base_link: mass None -> 0.001; geometry collision cylinder length=0.2 radius=0.1; visual cylinder length=0.2 radius=0.1
- link handle: mass None -> 0.001

Commit message: add all collision

File: urdf/kettle.urdf (robot description, URDF)
Before this commit: robot kettle, 4 links, 3 joints
Links:
- link base_link: mass 0.001 -> 0.1; geometry collision cylinder length=0.2 radius=0.95; visual cylinder length=0.2 radius=0.1
- link handle: mass 0.001 -> 0.02; geometry collision box size=0.02 0.185 0.01; visual box size=0.02 0.21 0.01
- link side1: geometry collision box size=0.02 0.01 0.1; visual box size=0.02 0.01 0.1
- link side2: geometry collision box size=0.02 0.01 0.1; visual box size=0.02 0.01 0.1
Joints:
- joint kettle_joint: limit lower=-1.57 upper=1.57 effort=1000000 velocity=10000 -> lower=-1.2 upper=1.2 effort=1000000 velocity=10000

Commit message: fixbug collision

File: urdf/kettle.urdf (robot description, URDF)
Before this commit: robot kettle, 4 links, 3 joints
Links:
- link base_link: geometry collision cylinder length=0.2 radius=0.095; visual cylinder length=0.2 radius=0.1

Commit message: gazebo setup fin

File: urdf/kettle.urdf (robot description, URDF)
Before this commit: robot kettle, 4 links, 3 joints
Links:
- link base_link: mass 0.1 -> 1.0
- link handle: mass 0.02 -> 0.2
